File: RX24T/base_board/rx24t_core.kicad_pcb (KiCad board)
At the start: 2 copper layers, 85 x 58 mm, 46 parts, among them P1 2X10, P10 2X10, P11 2X13, P2 2X13, P3 SPI-LCD, P4 SCI1, P5 SCI5, P6 APOWER, P7 SCI6, P8 I2C, P9 I2C, Q1 DMG3415U, SW1 3P-SW, SW2 RESET, U1 RX24T, U2 TCM809R, X1 10MHz

Commit message: update
Parts:
- L1, Q1, R1, R2, R3, U2: moved to B.Cu
- moved C9 25.0 mm to (149.9, 107.9)
- moved C3 23.6 mm to (143.1, 108.0)
- moved R1 21.4 mm to (123.5, 71.5), turned to 90 degrees
- moved R2 20.2 mm to (123.5, 77.4), turned to 90 degrees
- moved C7 18.6 mm to (161.9, 107.7)
- moved R3 17.7 mm to (123.1, 80.2)
- moved L1 15.6 mm to (125.4, 67.4), turned to 270 degrees
- moved C8 13.2 mm to (156.2, 108.0)
- moved C6 12.8 mm to (137.1, 107.7)
- moved Q1 11.5 mm to (126.4, 71.5)
- moved U2 10.5 mm to (126.5, 78.1)
- moved R6 9.52 mm to (181.2, 74.4)
- moved C1 3.63 mm to (116.3, 53.8)
- moved P1 2.54 mm to (122.9, 103.3)
- moved P2 2.54 mm to (150.8, 103.3)
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Routing:
- net /P01: track 0.00 -> 30.9 mm
- net /PE3: track 0.00 -> 28.8 mm
- net /PE4: track 0.00 -> 28.3 mm
- net /P41: track 0.00 -> 27.4 mm
- net /P43: track 0.00 -> 25.9 mm
- net /PE2: track 0.00 -> 25.5 mm
- net //RES: track 0.00 -> 25.1 mm
- net /P45: track 0.00 -> 24.5 mm
- net /PE0: track 0.00 -> 24.0 mm
- net /P42: track 0.00 -> 23.6 mm
- net /P47: track 0.00 -> 23.0 mm
- net /PD6: track 0.00 -> 22.6 mm
- net /P44: track 0.00 -> 22.1 mm
- net /PE1: track 0.00 -> 21.7 mm
- net /P51: track 0.00 -> 21.5 mm
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Other:
- board size 85 x 58 mm -> 85 x 55 mm
