File: rxprog/USB_CP2102N/USB_CP2102N.kicad_pcb (KiCad board)
At the start: 2 copper layers, 68.9 x 28.9 mm, 26 parts, among them J1 USB_B_Micro, J2 01x08, J3 02x03, J4 01x03, J5 01x06, U1 CP2102N, U2 NJU7223DL1-33

Commit message: Update: cleanup
Parts:
- moved TP1 3.86 mm to (139.7, 104.8)
Routing:
- net CTS: track 7.40 -> 81.2 mm, vias 0 -> 2
- net TXD: track 5.61 -> 67.9 mm, vias 0 -> 2
- net RTS: track 9.17 -> 64.9 mm, vias 0 -> 2
- net TXT: track 0.00 -> 53.6 mm, vias 0 -> 2
- net RXD: track 9.94 -> 60.1 mm, vias 0 -> 2
- net RXT: track 0.00 -> 47.9 mm, vias 0 -> 2
- net Net-(J2-Pad4): track 0.00 -> 45.8 mm, vias 0 -> 3
- net VDD: track 8.17 -> 40.3 mm, vias 2 -> 3
- net Net-(TP1-Pad1): track 0.00 -> 32.0 mm, vias 0 -> 1
- net +5V: track 69.0 -> 91.7 mm, vias 0 -> 1
- net Net-(J2-Pad6): track 0.00 -> 17.3 mm, vias 0 -> 1
- net Net-(J2-Pad5): track 0.00 -> 14.4 mm
- net Net-(J2-Pad3): track 0.00 -> 10.0 mm, vias 0 -> 1
- net GND: track 47.0 -> 52.7 mm, vias 5 -> 6
- added copper zone on B.Cu, net GND
- added copper zone on B.Cu, net Net-(C2-Pad1)
Other:
- board text added: "+3.3V"
- board text added: "+5V"
- board text added: "1:RXD"
- board text added: "2:TXD"
- board text added: "3:GND"
- board text added: "4:+V"
- board text added: "5:RTS"
- board text added: "6:CTS"
