File: DSOS_sample/DSO_FE/DSO_FE.kicad_sch (KiCad schematic)
At the start: 6 parts

Commit message: Update: FrontEnd
Parts:
- R? (x2): value R -> 1K
Other:
- sheet PreAmp ports: added CLK_REF_IN; removed REF_IN
- moved on the sheet: C?, R?, U?
