File: DSOS_sample/DSO_FE/FrontEnd.kicad_sch (KiCad schematic)
At the start: 32 parts

Commit message: Update: FrontEnd
Parts:
- added C? (x2): 4pF, symbol Akizuki:C
- added R? (x6): 100K, symbol Akizuki:R
- C? (x2): value 10pF -> 22pF
- C? (x2): value 22pF -> 100pF
- C? (x2): value 100pF -> 390pF
- GD? (x2): value GDT-SG75 -> GDT-SG90
- J? (x2): footprint (none) -> Connector_Coaxial:BNC_Amphenol_B6252HB-NPP3G-50_Horizontal
Connections:
- net +3V3: now also R?.1, R?.1, R?.1, R?.1
- net CH0_ACDC: now also R?.2
- net CH0_SA: now also R?.2
- net CH0_SB: now also R?.2
- net CH1_ACDC: now also R?.2
- net CH1_SA: now also R?.2
- net CH1_SB: now also R?.2
- net GND: now also R?.1, R?.1; no longer U?.1 (X4), U?.1 (X4), U?.2 (X6), U?.2 (X6), U?.4 (X7), U?.4 (X7), U?.5 (X5), U?.5 (X5), U?.6 (Inh), U?.6 (Inh), U?.9 (C), U?.9 (C)
- net GNDA: now also U?.1 (X4), U?.1 (X4), U?.2 (X6), U?.2 (X6), U?.4 (X7), U?.4 (X7), U?.5 (X5), U?.5 (X5), U?.6 (Inh), U?.6 (Inh), U?.9 (C), U?.9 (C)
- net at C?.1, C?.1, C?.2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: now also C?.1 (x2)
- net at C?.2, C?.2, R?.2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: now also C?.2 (x2)
Other:
- title: (none) -> フロントエンド
- moved on the sheet: GD?, J?, Q?
