File: DSOS_sample/DSO_FE/Power.kicad_sch (KiCad schematic)
At the start: 18 parts

Commit message: Update: FrontEnd
Parts:
- removed C?: 10uF, symbol Akizuki:C
- removed J?: USB_B_Micro, symbol Connector:USB_B_Micro
- removed U?: ADP2503, Package_CSP:LFCSP-WD-10-1EP_3x3mm_P0.5mm_EP1.64x2.38mm_ThermalVias, symbol Analog:ADP2503
- added BT?: Li3.7V, symbol Akizuki:BATTERY
- added C?: 10uF, symbol Akizuki:C
- added C?: 0.033uF, symbol Akizuki:C
- added C?: 3300pF, symbol Akizuki:C
- added D?: BLUE, symbol Device:LED_Filled
- added D?: SS2040FL, symbol Akizuki:Shotkey
- added J?: Barrel_Jack, symbol Connector:Barrel_Jack
- added JP?: Jumper_2_Bridged, symbol Jumper:Jumper_2_Bridged
- added M?: USB_LI_CHG, symbol Analog:USB_LI_CHG
- added R?: 10K, symbol Akizuki:R
- added R?: 330, symbol Akizuki:R
- added R?: 30K, symbol Akizuki:R
- added R?: 6.8K, symbol Akizuki:R
- added TP?: GNDA, symbol Connector:TestPoint
- added TP?: -5VA, symbol Connector:TestPoint
- added TP?: +5VA, symbol Connector:TestPoint
- added U?: ADP1613, Package_SO:MSOP-8-1EP_3x3mm_P0.65mm_EP1.68x1.88mm, symbol Analog:ADP1613
- L?: value 1.5uH -> 4.7uH
- PM?: footprint (none) -> KiCAD_lib:MAU106
Connections:
- net +5V: now also J?.1, JP?.2 (B), R?.2
- net +5VA: now also TP?.1
- net -5VA: now also TP?.1
- net GND: now also C?.1, C?.1, C?.1, D?.1 (K), J?.2, M?.1 (IN-), M?.3 (OUT-), R?.1, U?.4 (GND), U?.7 (FREQ)
- net GNDA: now also TP?.1
- net at C?.2, C?.2, JP?.2 (B): now also D?.1, R?.2
- net at L?.1: now also C?.2, M?.6 (OUT+), U?.6 (VIN)
- net at L?.2: now also D?.2, U?.5 (SW)
- new net: R?.1, R?.2, U?.2 (FB)
- new net: D?.2 (A), R?.1
- new net: C?.2, R?.1
- new net: R?.2, U?.1 (COMP)
- new net: C?.2, U?.8 (SS)
- new net: BT?.1 (+), M?.5 (BAT+)
- new net: BT?.2 (-), M?.4 (BAT-)
- new net: JP?.1 (A), M?.1 (IN-)
- no-connect marks 4 -> 0
Other:
- note added: "For Envision Kit Power"
- title: (none) -> 電源
- moved on the sheet: C?, J?, L?
