File: DSOS_sample/DSO_FE/PreAmp.kicad_sch (KiCad schematic)
At the start: 60 parts

Commit message: Update: FrontEnd
Parts:
- added RV? (x2): 500, symbol Device:R_Potentiometer
- added TP?: CH0, symbol Connector:TestPoint
- added TP?: CH1, symbol Connector:TestPoint
- R? (x2): value 5K -> 4.7K
Connections:
- net CH0_OUT: now also TP?.1
- net CH1_OUT: now also TP?.1
- net GNDA: now also RV?.2, RV?.2, RV?.3, RV?.3; no longer R?.1, R?.1
- net REF_IN renamed CLK_REF_IN
- new net: R?.1, RV?.1 (x2)
Other:
- title: (none) -> プリアンプ
