File: RX72M/MaxRX72M/LCD.kicad_sch (KiCad schematic)
At the start: 8 parts

Commit message: Update: cleanup
Parts:
- added MR?: 22, symbol Akizuki:MR
- added R?: 10K, symbol Akizuki:R
- added R?: 22, symbol Akizuki:R
Connections:
- net GND: now also CN?.29 (GND), CN?.3 (GND), CN?.36 (GND), R?.1
- net LCD_CLK: now also MR?.1
- net LCD_D0: now also MR?.4
- net LCD_D1: now also MR?.1
- net LCD_D10: now also MR?.2, MR?.4
- net LCD_D11: now also MR?.4
- net LCD_D12: now also MR?.1
- net LCD_D13: now also MR?.1, MR?.2
- net LCD_D14: now also MR?.2, MR?.3
- net LCD_D15: now also MR?.3, MR?.4
- net LCD_D2: now also MR?.1, MR?.2
- net LCD_D3: now also MR?.2, MR?.3
- net LCD_D4: now also MR?.3, MR?.4
- net LCD_D5: now also MR?.3
- net LCD_D6: now also MR?.4
- net LCD_D7: now also MR?.1
- net LCD_D8: now also MR?.2
- net LCD_D9: now also MR?.1, MR?.3
- net at CN?.30 (DCLK): now also MR?.8
- net at CN?.31 (DISP): now also MR?.7
- net at CN?.32 (HSYNC): now also MR?.6
- net at CN?.33 (VSYNC): now also MR?.5
- net at CN?.34 (DEN): now also R?.2
- new net LCD_DISP: MR?.2
- new net LCD_N0: MR?.4
- new net LCD_N2: MR?.3
- new net LCD_N3: R?.1, R?.2
