File: RX72M/MaxRX72M/MaxRX72M.kicad_sch (KiCad schematic)
At the start: 0 parts

Commit message: Update: cleanup
Other:
- sheet LCD ports: added LCD_CLK, LCD_DISP, LCD_N0, LCD_N2, LCD_N3; removed none
- sheet RX72M ports: added CRX0, CTX0, LCD_DISP, LCD_N0, NMI, USB_VBUSEN; removed none
Changed lines of the file:
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@@
+    (stroke (width 0) (type default) (color 0 0 0 0))
+  )
+  (wire (pts (xy 88.9 182.88) (xy 78.74 182.88))
     (stroke (width 0) (type default) (color 0 0 0 0))
   )
@@
     (stroke (width 0) (type default) (color 0 0 0 0))
   )
+  (wire (pts (xy 88.9 177.8) (xy 78.74 177.8))
+    (stroke (width 0) (type default) (color 0 0 0 0))
+  )
   (wire (pts (xy 78.74 143.51) (xy 88.9 143.51))
     (stroke (width 0) (type default) (color 0 0 0 0))
@@
     (stroke (width 0) (type default) (color 0 0 0 0))
   )
+  (wire (pts (xy 78.74 180.34) (xy 88.9 180.34))
+    (stroke (width 0) (type default) (color 0 0 0 0))
+  )
   (wire (pts (xy 54.61 168.91) (xy 43.18 168.91))
     (stroke (width 0) (type default) (color 0 0 0 0))
@@
     (stroke (width 0) (type default) (color 0 0 0 0))
   )
+  (wire (pts (xy 88.9 172.72) (xy 78.74 172.72))
+    (stroke (width 0) (type default) (color 0 0 0 0))
+  )
   (wire (pts (xy 54.61 173.99) (xy 43.18 173.99))
     (stroke (width 0) (type default) (color 0 0 0 0))
@@
   )
   (wire (pts (xy 43.18 113.03) (xy 54.61 113.03))
+    (stroke (width 0) (type default) (color 0 0 0 0))
+  )
+  (wire (pts (xy 78.74 175.26) (xy 88.9 175.26))
     (stroke (width 0) (type default) (color 0 0 0 0))
   )
@@
       (effects (font (size 1.27 1.27)) (justify right))
     )
-    (pin "LCD_CLK" input (at 78.74 121.92 0)
-      (effects (font (size 1.27 1.27)) (justify right))
-    )
-    (pin "LCD_N3" input (at 78.74 111.76 0)
-      (effects (font (size 1.27 1.27)) (justify right))
-    )
-    (pin "LCD_N2" input (at 78.74 114.3 0)
-      (effects (font (size 1.27 1.27)) (justify right))
-    )
-    (pin "USB_OVRCURA" input (at 78.74 59.69 0)
+    (pin "USB_OVRCURA" input (at 78.74 21.59 0)
+      (effects (font (size 1.27 1.27)) (justify right))
+    )
+    (pin "CRX0" input (at 78.74 107.95 0)
+      (effects (font (size 1.27 1.27)) (justify right))
+    )
+    (pin "CTX0" input (at 78.74 110.49 0)
+      (effects (font (size 1.27 1.27)) (justify right))
+    )
+    (pin "NMI" input (at 78.74 113.03 0)
+      (effects (font (size 1.27 1.27)) (justify right))
+    )
+    (pin "LCD_CLK" output (at 78.74 172.72 0)
+      (effects (font (size 1.27 1.27)) (justify right))
+    )
+    (pin "USB_VBUSEN" input (at 78.74 24.13 0)
+      (effects (font (size 1.27 1.27)) (justify right))
+    )
+    (pin "LCD_N0" output (at 78.74 175.26 0)
+      (effects (font (size 1.27 1.27)) (justify right))
+    )
+    (pin "LCD_N3" output (at 78.74 180.34 0)
+      (effects (font (size 1.27 1.27)) (justify right))
+    )
+    (pin "LCD_N2" output (at 78.74 177.8 0)
+      (effects (font (size 1.27 1.27)) (justify right))
+    )
+    (pin "LCD_DISP" output (at 78.74 182.88 0)
       (effects (font (size 1.27 1.27)) (justify right))
     )
@@
     )
   )
-  (sheet (at 127 92.71) (size 27.94 30.48) (fields_autoplaced)
+  (sheet (at 245.11 114.3) (size 27.94 30.48) (fields_autoplaced)
     (stroke (width 0) (type solid) (color 0 0 0 0))
     (fill (color 0 0 0 0.0000))
-    (property "Sheet name" "USB" (id 0) (at 127 91.9984 0)
+    (property "Sheet name" "USB" (id 0) (at 245.11 113.5884 0)
       (effects (font (size 1.27 1.27)) (justify left bottom))
     )
-    (property "Sheet file" "USB.kicad_sch" (id 1) (at 127 123.7746 0)
+    (property "Sheet file" "USB.kicad_sch" (id 1) (at 245.11 145.3646 0)
       (effects (font (size 1.27 1.27)) (justify left top))
     )
   )
-  (sheet (at 88.9 120.65) (size 21.59 71.12) (fields_autoplaced)
+  (sheet (at 88.9 120.65) (size 21.59 69.85) (fields_autoplaced)
     (stroke (width 0) (type solid) (color 0 0 0 0))
     (fill (color 0 0 0 0.0000))
@@
       (effects (font (size 1.27 1.27)) (justify left bottom))
     )
-    (property "Sheet file" "LCD.kicad_sch" (id 1) (at 88.9 192.3546 0)
+    (property "Sheet file" "LCD.kicad_sch" (id 1) (at 88.9 191.0846 0)
       (effects (font (size 1.27 1.27)) (justify left top))
     )
@@
     )
     (pin "LCD_D15" input (at 88.9 168.91 180)
+      (effects (font (size 1.27 1.27)) (justify left))
+    )
+    (pin "LCD_CLK" input (at 88.9 172.72 180)
+      (effects (font (size 1.27 1.27)) (justify left))
+    )
+    (pin "LCD_DISP" input (at 88.9 182.88 180)
+      (effects (font (size 1.27 1.27)) (justify left))
+    )
+    (pin "LCD_N2" input (at 88.9 177.8 180)
+      (effects (font (size 1.27 1.27)) (justify left))
+    )
+    (pin "LCD_N0" input (at 88.9 175.26 180)
+      (effects (font (size 1.27 1.27)) (justify left))
+    )
+    (pin "LCD_N3" input (at 88.9 180.34 180)
       (effects (font (size 1.27 1.27)) (justify left))
     )
@@
       (reference "#PWR?") (unit 1) (value "GND") (footprint "")
     )
+    (path "/00000000-0000-0000-0000-00005dc44928/15dc2039-0115-461d-8e4f-f5b966b00b41"
+      (reference "#PWR?") (unit 1) (value "GND") (footprint "")
+    )
     (path "/00000000-0000-0000-0000-00005dc44928/5ab70ec2-62a3-41fd-87e4-e9705e2957fa"
+      (reference "#PWR?") (unit 1) (value "GND") (footprint "")
+    )
+    (path "/00000000-0000-0000-0000-00005dba261f/b778e56d-aef3-48ca-a7ce-57459e070477"
+      (reference "#PWR?") (unit 1) (value "GNDA") (footprint "")
+    )
+    (path "/00000000-0000-0000-0000-00005dc44928/b9f86484-9e39-4063-bd16-ac90063f4b27"
       (reference "#PWR?") (unit 1) (value "GND") (footprint "")
     )
@@
       (reference "C?") (unit 1) (value "C") (footprint "")
     )
+    (path "/00000000-0000-0000-0000-00005dba261f/03c81442-c19f-418e-a99c-db7a87ead3cb"
+      (reference "C?") (unit 1) (value "0.1uF") (footprint "")
+    )
+    (path "/00000000-0000-0000-0000-00005dba261f/1669043a-cf51-4275-8a66-d30bc0d16cad"
+      (reference "C?") (unit 1) (value "0.1uF") (footprint "")
+    )
+    (path "/00000000-0000-0000-0000-00005dba261f/ca19150f-fd40-4f2c-b308-2bc56457d600"
+      (reference "C?") (unit 1) (value "10uF") (footprint "")
+    )
     (path "/00000000-0000-0000-0000-00005dc44928/28d79655-7732-4f4a-99bc-5b7897e8c970"
       (reference "CN?") (unit 1) (value "LCD_CAP_TOUCH") (footprint "")
@@
       (reference "D?") (unit 1) (value "6.8V") (footprint "")
     )
+    (path "/00000000-0000-0000-0000-00005dba261f/64e10260-191b-4601-a47c-7770f8f8080a"
+      (reference "FB?") (unit 1) (value "FB") (footprint "")
+    )
     (path "/00000000-0000-0000-0000-00005dc9399c/00000000-0000-0000-0000-00005dbf1a1c"
       (reference "J?") (unit 1) (value "J0011D21BNL") (footprint "")
     )
     (path "/00000000-0000-0000-0000-00005dc3479b/00000000-0000-0000-0000-00005dc3c34c"
-      (reference "J?") (unit 1) (value "USB_A") (footprint "")
+      (reference "J?") (unit 1) (value "HOST") (footprint "")
     )
     (path "/00000000-0000-0000-0000-00005dc340a2/00000000-0000-0000-0000-00005dc476e8"
       (reference "J?") (unit 1) (value "Micro_SD_Card_Det_Hirose_DM3AT") (footprint "")
     )
+    (path "/00000000-0000-0000-0000-00005dc3479b/7b38f0f1-c808-40fd-b2d6-944c19cfaf90"
+      (reference "J?") (unit 1) (value "DEVICE") (footprint "")
+    )
     (path "/00000000-0000-0000-0000-00005dc340a2/00000000-0000-0000-0000-00005dc7c168"
       (reference "JP?") (unit 1) (value "Jumper_2_Open") (footprint "")
@@
       (reference "MR?") (unit 1) (value "22") (footprint "")
     )
+    (path "/00000000-0000-0000-0000-00005dc44928/d7f3eb6a-aef9-4b1f-b472-f34135c0d830"
+      (reference "MR?") (unit 1) (value "22") (footprint "")
+    )
     (path "/00000000-0000-0000-0000-00005dc340a2/00000000-0000-0000-0000-00005dc4a789"
       (reference "R?") (unit 1) (value "22K") (footprint "")
@@
       (reference "R?") (unit 1) (value "4.7K") (footprint "")
     )
+    (path "/00000000-0000-0000-0000-00005dc44928/190cdc48-4dc8-4ac1-a58f-df57ed98ad9d"
+      (reference "R?") (unit 1) (value "10K") (footprint "")
+    )
+    (path "/00000000-0000-0000-0000-00005dc44928/a8b92650-4e44-4c78-989d-bd204f62f548"
+      (reference "R?") (unit 1) (value "22") (footprint "")
+    )
     (path "/00000000-0000-0000-0000-00005dc9399c/00000000-0000-0000-0000-00005dc93b7a"
