File: RX72M/MaxRX72M/Power.kicad_sch (KiCad schematic)
At the start: 15 parts

Commit message: Update: cleanup
Parts:
- added C? (x2): 0.1uF, symbol Akizuki:C
- added C?: 10uF, symbol Akizuki:CP
- added FB?: FB, symbol Akizuki:FB
Connections:
- net at C?.1: now also U?.14 (VCL); no longer U?.15 (VBATT)
- net at BT?.1 (+): now also U?.15 (VBATT); no longer U?.14 (VCL)
- net GNDA: now reaches U?.1 (AVSS0)
- net GNDA: now also U?.5 (AVSS1), C?.1, C?.1, C?.2
- net at U?.175 (AVCC0): now also U?.3 (AVCC1), C?.1, C?.2, C?.2, FB?.1
Other:
- moved on the sheet: BT?, C?, L?, U?
