File: RX72M/MaxRX72M/RX72M.kicad_sch (KiCad schematic)
At the start: 3 parts

Commit message: Update: cleanup
Connections:
- net LCD_N0: now reaches U?.52 (P13)
- net LCD_DISP: now reaches U?.13 (PJ3)
Changed lines of the file:
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@@
+    (stroke (width 0) (type default) (color 0 0 0 0))
+  )
+  (wire (pts (xy 259.08 38.1) (xy 254 38.1))
     (stroke (width 0) (type default) (color 0 0 0 0))
   )
@@
     (stroke (width 0) (type default) (color 0 0 0 0))
   )
+  (wire (pts (xy 58.42 63.5) (xy 53.34 63.5))
+    (stroke (width 0) (type default) (color 0 0 0 0))
+  )
   (wire (pts (xy 147.32 109.22) (xy 142.24 109.22))
     (stroke (width 0) (type default) (color 0 0 0 0))
@@
     (effects (font (size 1.27 1.27) (thickness 0.254) bold) (justify right))
   )
+  (hierarchical_label "LCD_DISP" (shape output) (at 259.08 38.1 0)
+    (effects (font (size 1.27 1.27) bold) (justify left))
+  )
   (hierarchical_label "ET_MDIO" (shape bidirectional) (at 52.07 106.68 180)
     (effects (font (size 1.27 1.27) (thickness 0.254) bold) (justify right))
@@
     (effects (font (size 1.27 1.27) (thickness 0.254) bold) (justify right))
   )
-  (hierarchical_label "LCD_N2" (shape input) (at 259.08 35.56 0)
-    (effects (font (size 1.27 1.27)) (justify left))
+  (hierarchical_label "LCD_N2" (shape output) (at 259.08 35.56 0)
+    (effects (font (size 1.27 1.27) (thickness 0.254) bold) (justify left))
   )
   (hierarchical_label "USB_OVRCURA" (shape input) (at 52.07 22.86 180)
@@
     (effects (font (size 1.27 1.27) (thickness 0.254) bold) (justify left))
   )
+  (hierarchical_label "LCD_N0" (shape output) (at 53.34 63.5 180)
+    (effects (font (size 1.27 1.27) (thickness 0.254) bold) (justify right))
+  )
   (hierarchical_label "ET_RXD0" (shape output) (at 142.24 66.04 180)
     (effects (font (size 1.27 1.27) (thickness 0.254) bold) (justify right))
@@
     (effects (font (size 1.27 1.27) (thickness 0.254) bold) (justify left))
   )
-  (hierarchical_label "LCD_N3" (shape input) (at 259.08 33.02 0)
-    (effects (font (size 1.27 1.27)) (justify left))
+  (hierarchical_label "LCD_N3" (shape output) (at 259.08 33.02 0)
+    (effects (font (size 1.27 1.27) (thickness 0.254) bold) (justify left))
   )
   (hierarchical_label "A4" (shape output) (at 142.24 91.44 180)
@@
     (effects (font (size 1.27 1.27) (thickness 0.254) bold) (justify left))
   )
-  (hierarchical_label "LCD_CLK" (shape input) (at 53.34 66.04 180)
+  (hierarchical_label "LCD_CLK" (shape output) (at 53.34 66.04 180)
     (effects (font (size 1.27 1.27) (thickness 0.254) bold) (justify right))
   )
@@
     (effects (font (size 1.27 1.27) (thickness 0.254) bold) (justify left))
   )
-  (hierarchical_label "USB_VBUSEN" (shape input) (at 53.34 71.12 180)
+  (hierarchical_label "USB_VBUSEN" (shape input) (at 52.07 25.4 180)
     (effects (font (size 1.27 1.27)) (justify right))
   )
