File: RX72M/MaxRX72M/SDIO.kicad_sch (KiCad schematic)
At the start: 12 parts

Commit message: Update: cleanup
Changed lines of the file:
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@@
-    (stroke (width 0) (type default) (color 0 0 0 0))
-  )
-  (wire (pts (xy 138.43 45.72) (xy 138.43 64.77))
     (stroke (width 0) (type default) (color 0 0 0 0))
   )
