File: RX72M/MaxRX72M/USB.kicad_sch (KiCad schematic)
At the start: 4 parts

Commit message: Update: cleanup
Parts:
- added J?: DEVICE, symbol Connector:USB_B_Mini
- J?: value USB_A -> HOST
Connections:
- net at D?.1 (K), J?.2 (D-), U?.55 (USB0_DM): now also J?.2 (D-)
- net at D?.1 (K), J?.3 (D+), U?.56 (USB0_DP): now also J?.3 (D+)
Changed lines of the file:
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@@
   (junction (at 105.41 124.46) (diameter 0) (color 0 0 0 0)
+  )
+  (wire (pts (xy 90.17 82.55) (xy 114.3 82.55))
+    (stroke (width 0) (type default) (color 0 0 0 0))
   )
   (wire (pts (xy 105.41 124.46) (xy 114.3 124.46))
@@
   )
   (wire (pts (xy 105.41 124.46) (xy 105.41 127))
+    (stroke (width 0) (type default) (color 0 0 0 0))
+  )
+  (wire (pts (xy 90.17 80.01) (xy 105.41 80.01))
     (stroke (width 0) (type default) (color 0 0 0 0))
   )
@@
     (stroke (width 0) (type default) (color 0 0 0 0))
   )
+  (wire (pts (xy 114.3 82.55) (xy 114.3 113.03))
+    (stroke (width 0) (type default) (color 0 0 0 0))
+  )
   (wire (pts (xy 105.41 120.65) (xy 105.41 124.46))
     (stroke (width 0) (type default) (color 0 0 0 0))
@@
     (stroke (width 0) (type default) (color 0 0 0 0))
   )
+  (wire (pts (xy 105.41 80.01) (xy 105.41 110.49))
+    (stroke (width 0) (type default) (color 0 0 0 0))
+  )
   (symbol (lib_id "Connector:USB_A") (at 82.55 110.49 0) (unit 1)
     (in_bom yes) (on_board yes)
     (property "Reference" "J?" (id 0) (at 83.9978 98.6282 0))
-    (property "Value" "USB_A" (id 1) (at 83.9978 100.9396 0))
+    (property "Value" "HOST" (id 1) (at 83.9978 100.9396 0))
     (property "Footprint" "" (id 2) (at 86.36 111.76 0)
       (effects (font (size 1.27 1.27)) hide)
@@
     (pin "57")
   )
+  (symbol (lib_id "Connector:USB_B_Mini") (at 82.55 80.01 0) (unit 1)
+    (in_bom yes) (on_board yes) (fields_autoplaced)
+    (property "Reference" "J?" (id 0) (at 82.55 68.6902 0))
+    (property "Value" "DEVICE" (id 1) (at 82.55 71.2271 0))
+    (property "Footprint" "" (id 2) (at 86.36 81.28 0)
+      (effects (font (size 1.27 1.27)) hide)
+    )
+    (property "Datasheet" "~" (id 3) (at 86.36 81.28 0)
+      (effects (font (size 1.27 1.27)) hide)
+    )
+    (pin "1")
+    (pin "2")
+    (pin "3")
+    (pin "4")
+    (pin "5")
+    (pin "6")
+  )
 )
