File: RX72T/RX72T_100_PGA_USB/rx72t_100_pga_usb.kicad_pcb (KiCad board)
At the start: 2 copper layers, 105 parts, among them J1 DA_OUT, J10 EMU_MODE, J11 SCI1, J12 5V_POW, J13 12V_POW, J14 CAN, J15 Micro_SD_Card_Det_Hirose_DM3AT, J17 MASTER, J18 I2C_B, J19 I2C_A, J2 GPTW_012, J20 RSPI, J21 SCI8, J22 SCI11, J23 SPI8, J24 SPI11, J25 RS-485 TERM, J26 RS-485, J27 MD, J3 GPTW_456, J4 EXT_DG0, J5 EXT_AN, J6 SCI1_POW, J7 UB, J8 EXT_DG1, J9 E1_E2_Lite, M1 BP5293-5, SW2 RESET, U2 SN65HVD230, U3 MIC2026-1BM, U4 MIC2026-1BM, U5 MAX3485, U6 RX72T_100_PGA_USB, X1 16MHz

Commit message: Update: cleanup
Parts:
- added J16: SLAVE, KiCAD_lib:HIROSE_MicroB_SMD, F.Cu at (51.3, 101.7)
- added J28: SER/RS-485, Connector_PinHeader_2.54mm:PinHeader_1x03_P2.54mm_Vertical, F.Cu at (160.5, 100.5)
- added J29: 5VIN, Connector_JST:JST_EH_B2B-EH-A_1x02_P2.50mm_Vertical, F.Cu at (124.3, 145.6)
- added U1: NJU7223DL1-33, Package_TO_SOT_SMD:TO-252-2, F.Cu at (124.3, 138.6)
- C1, C6: footprint Capacitor_THT:CP_Radial_D5.0mm_P2.00mm -> Capacitor_THT:CP_Radial_D4.0mm_P2.00mm
- C10, C16, C23, C24, C25, C26, C27, C29, C9: moved to B.Cu
- C30, C31: footprint Capacitor_THT:CP_Radial_D5.0mm_P2.00mm -> Capacitor_SMD:C_0805_2012Metric_Pad1.15x1.40mm_HandSolder
- C4, C7: footprint Capacitor_SMD:C_0805_2012Metric_Pad1.15x1.40mm_HandSolder -> Capacitor_THT:CP_Radial_D4.0mm_P2.00mm
- FB1, FB2: footprint Resistor_SMD:R_0805_2012Metric_Pad1.15x1.40mm_HandSolder -> Resistor_SMD:R_0603_1608Metric_Pad1.05x0.95mm_HandSolder
- X1: footprint Crystal:Crystal_SMD_HC49-SD_HandSoldering -> Crystal:Crystal_SMD_HC49-SD
- moved R16 94.9 mm to (142.7, 129.3), turned to 270 degrees
- moved J20 94.4 mm to (155.4, 141.1), turned to 180 degrees
- moved J23 92.9 mm to (160.5, 141.1), turned to 180 degrees
- moved R18 91.8 mm to (140.2, 129.3), turned to 270 degrees
- moved R13 91.8 mm to (144.6, 129.3), turned to 90 degrees
- moved R19 88.6 mm to (136.4, 129.3), turned to 270 degrees
- moved R21 88.4 mm to (150.3, 129.3), turned to 270 degrees
- moved R14 87.3 mm to (134.5, 129.3), turned to 270 degrees
- moved J15 85.6 mm to (144.0, 140.5)
- moved R17 85.3 mm to (148.4, 129.3), turned to 270 degrees
- moved R28 83.4 mm to (67.5, 87.8), turned to 180 degrees
- moved U3 82.9 mm to (141.4, 123.3)
- moved R20 82.3 mm to (138.3, 129.3), turned to 270 degrees
- moved J21 79.7 mm to (170.7, 133.5), turned to 180 degrees
- moved J24 76.2 mm to (160.5, 120.8), turned to 180 degrees
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Connections:
- C1 pad 1: GND -> +5V
- C1 pad 2: +5V -> GND
- C17 pad 1: GND -> Net-(C17-Pad1)
- C17 pad 2: Net-(C17-Pad2) -> GND
- C30 pad 1: GND -> +3V3
- C30 pad 2: +3V3 -> GND
- C31 pad 1: GNDA -> +3.3VA
- C31 pad 2: +3.3VA -> GNDA
- C4 pad 1: GND -> Net-(C2-Pad2)
- C4 pad 2: Net-(C2-Pad2) -> GND
- C6 pad 1: GND -> Net-(C6-Pad1)
- C6 pad 2: Net-(C6-Pad2) -> GND
- C7 pad 1: GND -> Net-(C5-Pad2)
- C7 pad 2: Net-(C5-Pad2) -> GND
- C8 pad 2: Net-(C6-Pad2) -> Net-(C6-Pad1)
- D1 pad 1: +12V -> Net-(C2-Pad2)
- D1 pad 2: Net-(C2-Pad2) -> +12V
- D2 pad 1: Net-(C6-Pad2) -> +5V
- D2 pad 2: +5V -> Net-(C6-Pad1)
- FB1 pad 1: (no net) -> +3V3
- FB1 pad 2: (no net) -> +3.3VA
- FB2 pad 1: (no net) -> GND
- FB2 pad 2: (no net) -> GNDA
- J12 pad 1: Net-(C6-Pad2) -> Net-(C6-Pad1)
- J17 pad 1: Net-(C17-Pad2) -> Net-(C17-Pad1)
- J22 pad 2: /RX72T/PA1_RXD11 -> Net-(J22-Pad2)
- J24 pad 1: /RX72T/PA1_RXD11 -> Net-(J22-Pad2)
- R9 pad 2: Net-(R9-Pad2) -> GND
- U3 pad 1: /SDC_IF/POW -> /RX72T/PA2_SCK11
- U4 pad 8: Net-(C17-Pad2) -> Net-(C17-Pad1)
- U5 pad 1: /RX72T/PA1_RXD11 -> Net-(J28-Pad3)
Routing:
- net GND: track 0.00 -> 682.8 mm, vias 0 -> 18
- net +3V3: track 0.00 -> 446.0 mm, vias 0 -> 20
- net +5V: track 0.00 -> 91.2 mm
- net GNDA: track 0.00 -> 80.5 mm, vias 0 -> 2
- net +3.3VA: track 0.00 -> 58.5 mm, vias 0 -> 2
- net Net-(C6-Pad1): track 0.00 -> 25.3 mm
- net Net-(C2-Pad2): track 0.00 -> 23.6 mm
- net Net-(C12-Pad2): track 0.00 -> 23.2 mm
- net Net-(C5-Pad2): track 0.00 -> 16.1 mm
- net Net-(C17-Pad1): track 0.00 -> 15.5 mm, vias 0 -> 1
- net /RX72T/PB2_SDA: track 0.00 -> 13.5 mm
- net /RX72T/PB1_SCL: track 0.00 -> 13.5 mm
- net Net-(C20-Pad2): track 0.00 -> 13.4 mm
- net Net-(C21-Pad2): track 0.00 -> 13.1 mm
- net Net-(F1-Pad2): track 0.00 -> 7.85 mm, vias 0 -> 1
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
Commit message: Update: cleanup
Parts:
- added H1: Hole, MountingHole:MountingHole_3.2mm_M3, F.Cu at (55.0, 145.0)
- added H2: Hole, MountingHole:MountingHole_3.2mm_M3, F.Cu at (55.0, 75.0)
- added H3: Hole, MountingHole:MountingHole_3.2mm_M3, F.Cu at (165.0, 75.0)
- added H4: Hole, MountingHole:MountingHole_3.2mm_M3, F.Cu at (165.0, 144.0)
- J15: value Micro_SD_Card_Det_Hirose_DM3AT -> MSD_Hirose_DM3AT
- moved C5 48.9 mm to (148.8, 115.7), turned to 180 degrees
- moved C7 47.7 mm to (143.3, 117.0)
- moved M1 35.6 mm to (144.0, 107.7), turned to 270 degrees
- moved J13 34.0 mm to (140.8, 110.0), turned to 0 degrees
- moved C2 31.1 mm to (148.8, 99.8), turned to 180 degrees
- moved J14 25.9 mm to (149.7, 72.5), turned to 0 degrees
- moved C4 24.9 mm to (143.3, 98.6)
- moved D1 21.8 mm to (149.2, 97.3)
- moved S1 18.3 mm to (148.4, 81.4), turned to 90 degrees
- moved J28 17.9 mm to (153.5, 117.0)
- moved S2 15.8 mm to (148.4, 77.6), turned to 90 degrees
- moved J26 9.67 mm to (166.8, 91.6)
- moved J25 9.44 mm to (162.4, 91.6)
- moved C11 9.38 mm to (142.9, 87.1)
- moved R11 9.38 mm to (146.8, 87.1)
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Routing:
- net GND: track 682.8 -> 950.1 mm, vias 18 -> 27
- net /PD3: track 0.00 -> 178.6 mm, vias 0 -> 1
- net /PD7: track 0.00 -> 176.7 mm, vias 0 -> 3
- net /PD4: track 0.00 -> 160.7 mm, vias 0 -> 1
- net +3V3: track 446.0 -> 598.3 mm, vias 20 -> 13
- net /PD5: track 0.00 -> 136.6 mm, vias 0 -> 2
- net /P00: track 0.00 -> 131.1 mm, vias 0 -> 1
- net /PE0: track 0.00 -> 116.8 mm, vias 0 -> 1
- net /RX72T/PA0_TXD11: track 0.00 -> 113.8 mm, vias 0 -> 1
- net /I2C_SPI_SCI/PB0: track 0.00 -> 111.8 mm, vias 0 -> 1
- net /I2C_SPI_SCI/MISO: track 2.60 -> 113.2 mm, vias 0 -> 2
- net /RX72T/PA5_RXD8: track 0.00 -> 105.5 mm, vias 0 -> 2
- net /PD6: track 0.00 -> 103.0 mm, vias 0 -> 2
- net /RX72T/PA4_TXD8: track 0.00 -> 98.9 mm, vias 0 -> 1
- net /PE3: track 0.00 -> 98.3 mm
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- added copper zone on B.Cu, net +3V3
- added copper zone on B.Cu, net GND
- added copper zone on F.Cu, net GND
Other:
- board outline added: 120 x 80 mm
- board text added: "RX72T PGA USB 100 Rev 1.00 https://github.com/hirakuni45"

Commit message: Update: cleanup
Other:
- net class Default removed
