File: RX140/RX140_board/Interface.kicad_sch (KiCad schematic)
At the start: 11 parts, among them SW1 RES, SW2 RUN/BOOT, X1 12MHz, X2 32.768KHz

Commit message: Update: cleanup
Parts:
- added C13: 0.1uF, symbol akizuki:C
- added D1: LED, symbol Device:LED
- added J1: SCI1, symbol Connector_Generic:Conn_02x03_Odd_Even
- added J1: SCI12, symbol Connector_Generic:Conn_02x03_Odd_Even
- added J2: I2C-A, symbol Connector_Generic:Conn_01x04
- added J3: I2C-B, symbol Connector_Generic:Conn_01x04
- added J6: EMU, symbol Connector_Generic:Conn_02x04_Odd_Even
- added J8: RSPI, symbol Connector_Generic:Conn_01x06
- added R3, R4, R5: 10K, symbol akizuki:R
- added R6: 1.5K, symbol akizuki:R
- added U3: SN65HVD230, Package_SO:SOP-8_3.76x4.96mm_P1.27mm, symbol analog:SN65HVD230
Connections:
- net GND: now also C13.2, J1.3 (Pin_3), J1.3 (Pin_3), J2.4 (Pin_4), J3.4 (Pin_4), J8.2 (Pin_2), U3.2 (GND)
- net VCC: now also C13.1, D1.2 (A), J1.4 (Pin_4), J1.4 (Pin_4), J2.3 (Pin_3), J3.3 (Pin_3), J8.1 (Pin_1), R3.2, R4.1, R5.1, U3.3 (Vcc)
- new net: D1.1 (K), R6.2
- new net CRXD0: U3.4 (R)
- new net CTXD0: U3.1 (D)
- new net LED: R6.1
- new net MISOA: J8.5 (Pin_5)
- new net MOSIA: J8.4 (Pin_4)
- new net NMI: R3.1
- new net RSPCKA: J8.3 (Pin_3)
- new net RXD1: J1.2 (Pin_2)
- new net RXD12: J1.2 (Pin_2)
- new net SCL0: J2.1 (Pin_1), J3.1 (Pin_1), R4.2
- new net SDA0: J2.2 (Pin_2), J3.2 (Pin_2), R5.2
- new net SSLA0: J8.6 (Pin_6)
- new net TXD1: J1.1 (Pin_1)
- new net TXD12: J1.1 (Pin_1)
- new net /CTS1: J1.5 (Pin_5)
- new net /CTS12: J1.5 (Pin_5)
- new net /RTS1: J1.6 (Pin_6)
- new net /RTS12: J1.6 (Pin_6)
Other:
- moved on the sheet: R2

Commit message: Update: cleanup
Parts:
- removed C13: 0.1uF, symbol akizuki:C
- removed U3: SN65HVD230, Package_SO:SOP-8_3.76x4.96mm_P1.27mm, symbol analog:SN65HVD230
- C8, C9: value 5pF -> 10pF
- U1: value ~ -> RX140

Commit message: Update: cleanup
Parts:
- C11: renamed from C6; footprint (none) -> Capacitor_SMD:C_0603_1608Metric_Pad1.08x0.95mm_HandSolder
- C12: renamed from C8; footprint (none) -> Capacitor_SMD:C_0603_1608Metric_Pad1.08x0.95mm_HandSolder
- C13: renamed from C9; footprint (none) -> Capacitor_SMD:C_0603_1608Metric_Pad1.08x0.95mm_HandSolder
- C14: renamed from C7; footprint (none) -> Capacitor_SMD:C_0603_1608Metric_Pad1.08x0.95mm_HandSolder
- D1: footprint (none) -> LED_SMD:LED_0603_1608Metric_Pad1.05x0.95mm_HandSolder
- J1: footprint (none) -> Connector_IDC:IDC-Header_2x03_P2.54mm_Vertical
- J10: renamed from J8; footprint (none) -> Connector_PinHeader_2.54mm:PinHeader_1x06_P2.54mm_Vertical
- J7: renamed from J6; footprint (none) -> Connector_IDC:IDC-Header_2x04_P2.54mm_Vertical
- J8: renamed from J2; footprint (none) -> Connector_PinHeader_2.54mm:PinHeader_1x04_P2.54mm_Vertical
- J9: renamed from J3; footprint (none) -> Connector_PinHeader_2.54mm:PinHeader_1x04_P2.54mm_Vertical
- R1: renamed from R2; footprint (none) -> Resistor_SMD:R_0603_1608Metric_Pad0.98x0.95mm_HandSolder
- R2: renamed from R1; footprint (none) -> Resistor_SMD:R_0603_1608Metric_Pad0.98x0.95mm_HandSolder
- R3: renamed from R4; value 10K -> 2K; footprint (none) -> Resistor_SMD:R_0603_1608Metric_Pad0.98x0.95mm_HandSolder
- R4: renamed from R5; value 10K -> 2K; footprint (none) -> Resistor_SMD:R_0603_1608Metric_Pad0.98x0.95mm_HandSolder
- R5: renamed from R3; footprint (none) -> Resistor_SMD:R_0603_1608Metric_Pad0.98x0.95mm_HandSolder
- R6: footprint (none) -> Resistor_SMD:R_0603_1608Metric_Pad0.98x0.95mm_HandSolder
- SW1: footprint (none) -> Button_Switch_THT:SW_PUSH_6mm
- SW2: footprint (none) -> Library:SW_3P_SPDT_Angled
- X1: renamed from X2; footprint Crystal:Crystal_SMD_HC49-SD_HandSoldering -> Crystal:Crystal_SMD_EuroQuartz_EQ161-2Pin_3.2x1.5mm_HandSoldering
- renumbered X1 to X2
Connections:
- net GND: now also J7.6 (Pin_6), J7.8 (Pin_8)
- net RXD1: now also J7.5 (Pin_5)
- net TXD1: now also J7.7 (Pin_7)
- net VCC: now also J7.2 (Pin_2)
- net at R2.1, SW1.2, U1.6 (~{RES}): now also J7.1 (Pin_1)
- net at J7.3 (Pin_3): now also R1.2, U1.3 (PG7/MD)
- net /RTS12 renamed PE0
- no-connect marks 0 -> 1
Other:
- moved on the sheet: C11, C12, C13, C14, J7, R1, R2, SW1, SW2, U1A, X1, X2
