File: RX140/RX140_board/Power.kicad_sch (KiCad schematic)
At the start: 9 parts

Commit message: Update: cleanup
Parts:
- added C11, C15: 0.1uF, symbol akizuki:C
- added C12, C14: 0.01uF, symbol akizuki:C
- added FB3: FB, symbol akizuki:FB
- added J4: POWER, symbol Connector_Generic:Conn_01x02
- added J5: AUDIO, symbol Connector_Generic:Conn_01x04
- C2, C3, C4: value 104 -> 0.1uF
Connections:
- net GND: now also C15.1, J4.2 (Pin_2)
- net GNDA: now also C11.1, C12.1, C14.2, J5.4 (Pin_4)
- net VCC: now also C15.2, FB3.2, J4.1 (Pin_1)
- net at C4.1, FB2.1, U1.62 (AVCC0): now also C14.1, J5.1 (Pin_1)
- net at U1.61 (VREFH0/PJ6): now also C11.2, C12.2, FB3.1
- new net DA0: J5.2 (Pin_2)
- new net DA1: J5.3 (Pin_3)
Other:
- moved on the sheet: FB2

Commit message: Update: cleanup
Parts:
- U1: value ~ -> RX140
Changed lines of the file:
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@@
   )
   (symbol (lib_id "renesas:RX140_64") (at 68.58 86.36 0) (unit 2)
-    (in_bom yes) (on_board yes) (dnp no) (fields_autoplaced)
-    (property "Reference" "U1" (at 50.7285 85.4489 0)
+    (in_bom yes) (on_board yes) (dnp no)
+    (property "Reference" "U1" (at 50.8 69.85 0)
       (effects (font (size 1.27 1.27)))
     )
-    (property "Value" "~" (at 68.58 72.39 0)
+    (property "Value" "RX140" (at 49.53 72.39 0)
       (effects (font (size 1.27 1.27)))
     )

Commit message: Update: cleanup
Parts:
- removed J5: AUDIO, symbol Connector_Generic:Conn_01x04
- added J16: GND, TestPoint:TestPoint_Bridge_Pitch2.54mm_Drill1.0mm, symbol Connector_Generic:Conn_01x01
- added J4: D/A, Connector_PinHeader_2.54mm:PinHeader_1x05_P2.54mm_Vertical, symbol Connector_Generic:Conn_01x05
- C1: renamed from C2; footprint (none) -> Capacitor_SMD:C_0603_1608Metric_Pad1.08x0.95mm_HandSolder
- C10: renamed from C11; footprint (none) -> Capacitor_SMD:C_0603_1608Metric_Pad1.08x0.95mm_HandSolder
- C2: renamed from C3; footprint (none) -> Capacitor_SMD:C_0603_1608Metric_Pad1.08x0.95mm_HandSolder
- C3: renamed from C10; footprint (none) -> Capacitor_SMD:C_0603_1608Metric_Pad1.08x0.95mm_HandSolder
- C4: renamed from C1; footprint (none) -> Capacitor_SMD:C_0603_1608Metric_Pad1.08x0.95mm_HandSolder
- C5: renamed from C14; footprint (none) -> Capacitor_SMD:C_0603_1608Metric_Pad1.08x0.95mm_HandSolder
- C6: renamed from C4; footprint (none) -> Capacitor_SMD:C_0603_1608Metric_Pad1.08x0.95mm_HandSolder
- C7: renamed from C15; footprint (none) -> Capacitor_SMD:C_0603_1608Metric_Pad1.08x0.95mm_HandSolder
- C8: renamed from C5; footprint (none) -> Capacitor_SMD:C_0603_1608Metric_Pad1.08x0.95mm_HandSolder
- C9: renamed from C12; footprint (none) -> Capacitor_SMD:C_0603_1608Metric_Pad1.08x0.95mm_HandSolder
- FB1, FB2, FB3: footprint (none) -> Resistor_SMD:R_0603_1608Metric_Pad0.98x0.95mm_HandSolder
- J3: renamed from J4; footprint (none) -> Connector_PinHeader_2.54mm:PinHeader_1x02_P2.54mm_Vertical
Connections:
- net DA0: now also J4.2 (Pin_2)
- net DA1: now also J4.3 (Pin_3)
- net GND: now also J16.1 (Pin_1)
- net GNDA: now also J4.4 (Pin_4), J4.5 (Pin_5)
- net VDD: now reaches C5.1, C6.1, FB2.1, U1.62 (AVCC0)
- net VDD: now also J4.1 (Pin_1)
Other:
- moved on the sheet: C7, C8
