File: RX140/RX140_board/RX140_board.kicad_sch (KiCad schematic)
At the start: 1 part

Commit message: Update: cleanup
Connections:
- net DA0: now reaches U1.1 (P03)
- net NMI: now reaches U1.11 (P35)
- net /RTS1: now reaches U1.13 (P31)
- net RXD1: now reaches U1.14 (P30)
- net TXD1: now reaches U1.16 (P26)
- net SDA0: now reaches U1.17 (P17)
- net SCL0: now reaches U1.18 (P16)
- net LED: now reaches U1.19 (P15)
- net /CTS1: now reaches U1.20 (P14)
- net CRXD0: now reaches U1.25 (P55)
- net CTXD0: now reaches U1.26 (P54)
- net DA1: now reaches U1.63 (P05)
- net MISOA: now reaches U1.27 (PC7)
- net MOSIA: now reaches U1.28 (PC6)
- net RSPCKA: now reaches U1.29 (PC5)
- net SSLA0: now reaches U1.30 (PC4)
- net /CTS12: now reaches U1.48 (PE3)
- net RXD12: now reaches U1.49 (PE2)
- net TXD12: now reaches U1.50 (PE1)
Changed lines of the file:
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@@
 (kicad_sch (version 20230121) (generator eeschema)
   (paper "A4")
+  (wire (pts (xy 165.1 62.23) (xy 172.72 62.23))
+    (stroke (width 0) (type default))
+  )
+  (wire (pts (xy 50.8 67.31) (xy 55.88 67.31))
+    (stroke (width 0) (type default))
+  )
+  (wire (pts (xy 50.8 64.77) (xy 55.88 64.77))
+    (stroke (width 0) (type default))
+  )
+  (wire (pts (xy 50.8 41.91) (xy 55.88 41.91))
+    (stroke (width 0) (type default))
+  )
+  (wire (pts (xy 165.1 59.69) (xy 172.72 59.69))
+    (stroke (width 0) (type default))
+  )
+  (wire (pts (xy 165.1 118.11) (xy 171.45 118.11))
+    (stroke (width 0) (type default))
+  )
+  (wire (pts (xy 50.8 105.41) (xy 55.88 105.41))
+    (stroke (width 0) (type default))
+  )
+  (wire (pts (xy 165.1 57.15) (xy 172.72 57.15))
+    (stroke (width 0) (type default))
+  )
+  (wire (pts (xy 165.1 120.65) (xy 171.45 120.65))
+    (stroke (width 0) (type default))
+  )
+  (wire (pts (xy 86.36 92.71) (xy 88.9 92.71))
+    (stroke (width 0) (type default))
+  )
+  (wire (pts (xy 86.36 90.17) (xy 88.9 90.17))
+    (stroke (width 0) (type default))
+  )
+  (wire (pts (xy 50.8 72.39) (xy 55.88 72.39))
+    (stroke (width 0) (type default))
+  )
+  (wire (pts (xy 50.8 34.29) (xy 55.88 34.29))
+    (stroke (width 0) (type default))
+  )
+  (wire (pts (xy 50.8 95.25) (xy 55.88 95.25))
+    (stroke (width 0) (type default))
+  )
+  (wire (pts (xy 165.1 115.57) (xy 171.45 115.57))
+    (stroke (width 0) (type default))
+  )
+  (wire (pts (xy 165.1 123.19) (xy 171.45 123.19))
+    (stroke (width 0) (type default))
+  )
+  (wire (pts (xy 50.8 69.85) (xy 55.88 69.85))
+    (stroke (width 0) (type default))
+  )
+  (wire (pts (xy 50.8 107.95) (xy 55.88 107.95))
+    (stroke (width 0) (type default))
+  )
+  (wire (pts (xy 50.8 118.11) (xy 55.88 118.11))
+    (stroke (width 0) (type default))
+  )
+  (global_label "{slash}CTS1" (shape input) (at 50.8 64.77 180) (fields_autoplaced)
+    (effects (font (size 1.27 1.27)) (justify right))
+    (property "Intersheetrefs" "${INTERSHEET_REFS}" (at 41.9071 64.77 0)
+      (effects (font (size 1.27 1.27)) (justify right) hide)
+    )
+  )
+  (global_label "MISOA" (shape input) (at 171.45 123.19 0) (fields_autoplaced)
+    (effects (font (size 1.27 1.27)) (justify left))
+    (property "Intersheetrefs" "${INTERSHEET_REFS}" (at 180.0406 123.19 0)
+      (effects (font (size 1.27 1.27)) (justify left) hide)
+    )
+  )
+  (global_label "DA1" (shape input) (at 50.8 41.91 180) (fields_autoplaced)
+    (effects (font (size 1.27 1.27)) (justify right))
+    (property "Intersheetrefs" "${INTERSHEET_REFS}" (at 44.3261 41.91 0)
+      (effects (font (size 1.27 1.27)) (justify right) hide)
+    )
+  )
+  (global_label "RXD1" (shape input) (at 50.8 105.41 180) (fields_autoplaced)
+    (effects (font (size 1.27 1.27)) (justify right))
+    (property "Intersheetrefs" "${INTERSHEET_REFS}" (at 42.9352 105.41 0)
+      (effects (font (size 1.27 1.27)) (justify right) hide)
+    )
+  )
+  (global_label "LED" (shape input) (at 50.8 67.31 180) (fields_autoplaced)
+    (effects (font (size 1.27 1.27)) (justify right))
+    (property "Intersheetrefs" "${INTERSHEET_REFS}" (at 44.4471 67.31 0)
+      (effects (font (size 1.27 1.27)) (justify right) hide)
+    )
+  )
+  (global_label "CRXD0" (shape input) (at 88.9 92.71 0) (fields_autoplaced)
+    (effects (font (size 1.27 1.27)) (justify left))
+    (property "Intersheetrefs" "${INTERSHEET_REFS}" (at 98.0348 92.71 0)
+      (effects (font (size 1.27 1.27)) (justify left) hide)
+    )
+  )
+  (global_label "TXD12" (shape input) (at 172.72 57.15 0) (fields_autoplaced)
+    (effects (font (size 1.27 1.27)) (justify left))
+    (property "Intersheetrefs" "${INTERSHEET_REFS}" (at 181.4919 57.15 0)
+      (effects (font (size 1.27 1.27)) (justify left) hide)
+    )
+  )
+  (global_label "{slash}RTS1" (shape input) (at 50.8 107.95 180) (fields_autoplaced)
+    (effects (font (size 1.27 1.27)) (justify right))
+    (property "Intersheetrefs" "${INTERSHEET_REFS}" (at 41.9071 107.95 0)
+      (effects (font (size 1.27 1.27)) (justify right) hide)
+    )
+  )
+  (global_label "{slash}CTS12" (shape input) (at 172.72 62.23 0) (fields_autoplaced)
+    (effects (font (size 1.27 1.27)) (justify left))
+    (property "Intersheetrefs" "${INTERSHEET_REFS}" (at 182.8224 62.23 0)
+      (effects (font (size 1.27 1.27)) (justify left) hide)
+    )
+  )
+  (global_label "RXD12" (shape input) (at 172.72 59.69 0) (fields_autoplaced)
+    (effects (font (size 1.27 1.27)) (justify left))
+    (property "Intersheetrefs" "${INTERSHEET_REFS}" (at 181.7943 59.69 0)
+      (effects (font (size 1.27 1.27)) (justify left) hide)
+    )
+  )
+  (global_label "RSPCKA" (shape input) (at 171.45 118.11 0) (fields_autoplaced)
+    (effects (font (size 1.27 1.27)) (justify left))
+    (property "Intersheetrefs" "${INTERSHEET_REFS}" (at 181.7339 118.11 0)
+      (effects (font (size 1.27 1.27)) (justify left) hide)
+    )
+  )
+  (global_label "SSLA0" (shape input) (at 171.45 115.57 0) (fields_autoplaced)
+    (effects (font (size 1.27 1.27)) (justify left))
+    (property "Intersheetrefs" "${INTERSHEET_REFS}" (at 180.101 115.57 0)
+      (effects (font (size 1.27 1.27)) (justify left) hide)
+    )
+  )
+  (global_label "SDA0" (shape input) (at 50.8 72.39 180) (fields_autoplaced)
+    (effects (font (size 1.27 1.27)) (justify right))
+    (property "Intersheetrefs" "${INTERSHEET_REFS}" (at 43.1166 72.39 0)
+      (effects (font (size 1.27 1.27)) (justify right) hide)
+    )
+  )
+  (global_label "TXD1" (shape input) (at 50.8 95.25 180) (fields_autoplaced)
+    (effects (font (size 1.27 1.27)) (justify right))
+    (property "Intersheetrefs" "${INTERSHEET_REFS}" (at 43.2376 95.25 0)
+      (effects (font (size 1.27 1.27)) (justify right) hide)
+    )
+  )
+  (global_label "DA0" (shape input) (at 50.8 34.29 180) (fields_autoplaced)
+    (effects (font (size 1.27 1.27)) (justify right))
+    (property "Intersheetrefs" "${INTERSHEET_REFS}" (at 44.3261 34.29 0)
+      (effects (font (size 1.27 1.27)) (justify right) hide)
+    )
+  )
+  (global_label "SCL0" (shape input) (at 50.8 69.85 180) (fields_autoplaced)
+    (effects (font (size 1.27 1.27)) (justify right))
+    (property "Intersheetrefs" "${INTERSHEET_REFS}" (at 43.1771 69.85 0)
+      (effects (font (size 1.27 1.27)) (justify right) hide)
+    )
+  )
+  (global_label "MOSIA" (shape input) (at 171.45 120.65 0) (fields_autoplaced)
+    (effects (font (size 1.27 1.27)) (justify left))
+    (property "Intersheetrefs" "${INTERSHEET_REFS}" (at 180.0406 120.65 0)
+      (effects (font (size 1.27 1.27)) (justify left) hide)
+    )
+  )
+  (global_label "NMI" (shape input) (at 50.8 118.11 180) (fields_autoplaced)
+    (effects (font (size 1.27 1.27)) (justify right))
+    (property "Intersheetrefs" "${INTERSHEET_REFS}" (at 44.5075 118.11 0)
+      (effects (font (size 1.27 1.27)) (justify right) hide)
+    )
+  )
+  (global_label "CTXD0" (shape input) (at 88.9 90.17 0) (fields_autoplaced)
+    (effects (font (size 1.27 1.27)) (justify left))
+    (property "Intersheetrefs" "${INTERSHEET_REFS}" (at 97.7324 90.17 0)
+      (effects (font (size 1.27 1.27)) (justify left) hide)
+    )
+  )
   (symbol (lib_id "renesas:RX140_64") (at 71.12 76.2 0) (unit 3)
     (in_bom yes) (on_board yes) (dnp no) (fields_autoplaced)

Commit message: Update: cleanup
Parts:
- U1: value ~ -> RX140
Connections:
- net CRXD0: no longer names the net of U1.25 (P55)
- net CTXD0: no longer names the net of U1.26 (P54)
Other:
- added sheet CH340 Serial USB (ch340_if.kicad_sch)
Changed lines of the file:
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@@
-    (stroke (width 0) (type default))
-  )
-  (wire (pts (xy 86.36 92.71) (xy 88.9 92.71))
-    (stroke (width 0) (type default))
-  )
-  (wire (pts (xy 86.36 90.17) (xy 88.9 90.17))
     (stroke (width 0) (type default))
   )
@@
     )
   )
-  (global_label "CRXD0" (shape input) (at 88.9 92.71 0) (fields_autoplaced)
-    (effects (font (size 1.27 1.27)) (justify left))
-    (property "Intersheetrefs" "${INTERSHEET_REFS}" (at 98.0348 92.71 0)
-      (effects (font (size 1.27 1.27)) (justify left) hide)
-    )
-  )
   (global_label "TXD12" (shape input) (at 172.72 57.15 0) (fields_autoplaced)
     (effects (font (size 1.27 1.27)) (justify left))
@@
     )
   )
-  (global_label "CTXD0" (shape input) (at 88.9 90.17 0) (fields_autoplaced)
-    (effects (font (size 1.27 1.27)) (justify left))
-    (property "Intersheetrefs" "${INTERSHEET_REFS}" (at 97.7324 90.17 0)
-      (effects (font (size 1.27 1.27)) (justify left) hide)
-    )
-  )
   (symbol (lib_id "renesas:RX140_64") (at 71.12 76.2 0) (unit 3)
-    (in_bom yes) (on_board yes) (dnp no) (fields_autoplaced)
-    (property "Reference" "U1" (at 71.12 23.1681 0)
+    (in_bom yes) (on_board yes) (dnp no)
+    (property "Reference" "U1" (at 71.12 20.32 0)
       (effects (font (size 1.27 1.27)))
     )
-    (property "Value" "~" (at 71.12 62.23 0)
+    (property "Value" "RX140" (at 71.12 22.86 0)
       (effects (font (size 1.27 1.27)))
     )
@@
   )
   (symbol (lib_id "renesas:RX140_64") (at 149.86 74.93 0) (unit 4)
-    (in_bom yes) (on_board yes) (dnp no) (fields_autoplaced)
-    (property "Reference" "U1" (at 149.86 23.1681 0)
+    (in_bom yes) (on_board yes) (dnp no)
+    (property "Reference" "U1" (at 149.86 20.32 0)
       (effects (font (size 1.27 1.27)))
     )
-    (property "Value" "~" (at 149.86 60.96 0)
+    (property "Value" "RX140" (at 149.86 22.86 0)
       (effects (font (size 1.27 1.27)))
     )
@@
     )
   )
-  (sheet (at 62.23 157.48) (size 41.91 20.32) (fields_autoplaced)
+  (sheet (at 118.11 153.67) (size 41.91 20.32) (fields_autoplaced)
     (stroke (width 0.1524) (type solid))
     (fill (color 0 255 255 1.0000))
-    (property "Sheetname" "Power" (at 62.23 156.7684 0)
+    (property "Sheetname" "Power" (at 118.11 152.9584 0)
       (effects (font (size 1.27 1.27)) (justify left bottom))
     )
-    (property "Sheetfile" "Power.kicad_sch" (at 62.23 178.3846 0)
+    (property "Sheetfile" "Power.kicad_sch" (at 118.11 174.5746 0)
       (effects (font (size 1.27 1.27)) (justify left top))
     )
@@
       )
     )
+  )
+  (sheet (at 62.23 152.4) (size 40.64 21.59) (fields_autoplaced)
+    (stroke (width 0.1524) (type solid))
+    (fill (color 0 255 255 1.0000))
+    (property "Sheetname" "CH340 Serial USB" (at 62.23 151.6884 0)
+      (effects (font (size 1.27 1.27)) (justify left bottom))
+    )
+    (property "Sheetfile" "ch340_if.kicad_sch" (at 62.23 174.5746 0)
+      (effects (font (size 1.27 1.27)) (justify left top))
+    )
+    (instances
+      (project "RX140_board"
+        (path "/1ba7daaa-0b3e-4d88-b450-d41f3b2cc6e9" (page "4"))
+      )
+    )

Commit message: Update: cleanup
Parts:
- added J1: PIN-A, Connector_PinHeader_2.54mm:PinHeader_1x30_P2.54mm_Vertical, symbol Connector_Generic:Conn_01x30
- added J2: PIN-B, Connector_PinHeader_2.54mm:PinHeader_1x30_P2.54mm_Vertical, symbol Connector_Generic:Conn_01x30
- added NT1: TIE_RXD, Connector_PinHeader_2.54mm:PinHeader_1x02_P2.54mm_Vertical, symbol Device:NetTie_2
- added NT2: TIE_TXD, Connector_PinHeader_2.54mm:PinHeader_1x02_P2.54mm_Vertical, symbol Device:NetTie_2
Connections:
- net DA0: now also J1.27 (Pin_27)
- net DA1: now also J1.28 (Pin_28)
- net LED: now also J1.8 (Pin_8)
- net MISOA: now also J2.17 (Pin_17)
- net MOSIA: now also J2.16 (Pin_16)
- net NMI: now also J1.16 (Pin_16)
- net RSPCKA: now also J2.15 (Pin_15)
- net RXD1: now also J1.13 (Pin_13), NT1.2
- net RXD12: now also J2.21 (Pin_21)
- net SCL0: now also J1.9 (Pin_9)
- net SDA0: now also J1.10 (Pin_10)
- net SSLA0: now also J2.14 (Pin_14)
- net TXD1: now also J1.11 (Pin_11), NT2.2
- net TXD12: now also J2.20 (Pin_20)
- net /CTS1: now also J1.7 (Pin_7)
- net /CTS12: now also J2.22 (Pin_22)
- net /RTS1: now also J1.14 (Pin_14)
- net P32: now reaches U1.12 (P32)
- net P32: now also J1.15 (Pin_15)
- net P27: now reaches U1.15 (P27)
- net P27: now also J1.12 (Pin_12)
- net P55: now reaches U1.25 (P55)
- net P55: now also J1.3 (Pin_3)
- net P54: now reaches U1.26 (P54)
- net P54: now also J1.2 (Pin_2)
- net P47: now reaches U1.52 (P47)
- net P47: now also J1.25 (Pin_25)
- net P46: now reaches U1.53 (P46)
- net P46: now also J1.24 (Pin_24)
- net P45: now reaches U1.54 (P45)
- net P45: now also J1.23 (Pin_23)
- net P44: now reaches U1.55 (P44)
- net P44: now also J1.22 (Pin_22)
- net P43: now reaches U1.56 (P43)
- net P43: now also J1.21 (Pin_21)
- net P42: now reaches U1.57 (P42)
- net P42: now also J1.20 (Pin_20)
- net P41: now reaches U1.58 (P41)
- net P41: now also J1.19 (Pin_19)
- net P40: now reaches U1.60 (P40)
- net P40: now also J1.18 (Pin_18)
- net PH3: now reaches U1.21 (PH3)
- net PH3: now also J2.29 (Pin_29)
- net PH2: now reaches U1.22 (PH2)
- net PH2: now also J2.28 (Pin_28)
- net PH1: now reaches U1.23 (PH1)
- net PH1: now also J2.27 (Pin_27)
- net PH0: now reaches U1.24 (PH0)
- net PH0: now also J2.26 (Pin_26)
- net PC3: now reaches U1.31 (PC3)
- net PC3: now also J2.13 (Pin_13)
- net PC2: now reaches U1.32 (PC2)
- net PC2: now also J2.12 (Pin_12)
- net PB7: now reaches U1.33 (PB7/PC1)
- net PB7: now also J2.11 (Pin_11)
- net PB6: now reaches U1.34 (PB6/PC0)
- net PB6: now also J2.10 (Pin_10)
- net PB5: now reaches U1.35 (PB5)
- net PB5: now also J2.9 (Pin_9)
- net PB3: now reaches U1.36 (PB3)
- net PB3: now also J2.8 (Pin_8)
- net PB1: now reaches U1.37 (PB1)
- net PB1: now also J2.7 (Pin_7)
- net PB0: now reaches U1.39 (PB0)
- net PB0: now also J2.6 (Pin_6)
- net PA6: now reaches U1.41 (PA6)
- net PA6: now also J2.4 (Pin_4)
- net PA4: now reaches U1.42 (PA4)
- net PA4: now also J2.3 (Pin_3)
- net PA3: now reaches U1.43 (PA3)
- net PA3: now also J2.2 (Pin_2)
- net PA1: now reaches U1.44 (PA1)
- net PA1: now also J1.5 (Pin_5)
- net PA0: now reaches U1.45 (PA0)
- net PA0: now also J1.4 (Pin_4)
- net PE5: now reaches U1.46 (PE5)
- net PE5: now also J2.24 (Pin_24)
- net PE4: now reaches U1.47 (PE4)
- net PE4: now also J2.23 (Pin_23)
- net PE0: now reaches U1.51 (PE0)
- net PE0: now also J2.19 (Pin_19)
- new net CH340 Serial USB/RXD: NT2.1
- new net CH340 Serial USB/TXD: NT1.1
- new net GND: J1.30 (Pin_30), J1.6 (Pin_6), J2.18 (Pin_18), J2.30 (Pin_30), J2.5 (Pin_5)
- new net GNDA: J1.26 (Pin_26)
- new net VCC: J1.1 (Pin_1), J1.29 (Pin_29), J2.1 (Pin_1), J2.25 (Pin_25)
- new net VDD: J1.17 (Pin_17)
Other:
- sheet CH340 Serial USB ports: added RXD, TXD; removed none
- moved on the sheet: U1C, U1D
