File: RX140/RX140_board/ch340_if.kicad_sch (KiCad schematic)
At the start: 9 parts, among them J9 USB_B_Micro, U2 CH340K, U3 NJU7223DL1-33

Commit message: Update: cleanup
Parts:
- added J12: 3.3V_CON, Connector_PinHeader_2.54mm:PinHeader_1x02_P2.54mm_Vertical, symbol Connector_Generic:Conn_01x02
- added J13: Serial, Connector_IDC:IDC-Header_2x03_P2.54mm_Vertical, symbol Connector_Generic:Conn_02x03_Odd_Even
- added J14: /DTR, Connector_PinHeader_2.54mm:PinHeader_1x02_P2.54mm_Vertical, symbol Connector_Generic:Conn_01x02
- added J15: 5/3.3, Connector_PinHeader_2.54mm:PinHeader_1x03_P2.54mm_Vertical, symbol Connector_Generic:Conn_01x03
- C15: renamed from C13; footprint (none) -> Capacitor_SMD:C_0603_1608Metric_Pad1.08x0.95mm_HandSolder
- C16: renamed from C17; footprint (none) -> Capacitor_SMD:C_0603_1608Metric_Pad1.08x0.95mm_HandSolder
- C17: renamed from C16; footprint (none) -> Capacitor_SMD:C_0603_1608Metric_Pad1.08x0.95mm_HandSolder
- C18: footprint (none) -> Capacitor_SMD:C_0603_1608Metric_Pad1.08x0.95mm_HandSolder
- C19: value 0.1uF -> 1uF; footprint (none) -> Capacitor_SMD:C_0603_1608Metric_Pad1.08x0.95mm_HandSolder
- F1: footprint (none) -> Capacitor_THT:C_Disc_D4.3mm_W1.9mm_P5.00mm
- J11: renamed from J9; footprint (none) -> Library:USB_MICRO_B-HIROSE-ZX62R-B-5P
- U2: renamed from U3; footprint TO_SOT_Packages_SMD:TO-252-2 -> Package_TO_SOT_SMD:TO-252-2
- renumbered U2 to U3
Connections:
- net GND: now also J13.3 (Pin_3), J14.2 (Pin_2)
- net RXD: now also J13.1 (Pin_1)
- net TXD: now also J13.2 (Pin_2)
- net VCC: now also J12.2 (Pin_2); no longer C19.2, U2.1 (Vout)
- net at C16.2, C17.2, C18.2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: now also J15.1 (Pin_1)
- net /CTS: no longer names the net of U3.5 (CTS#)
- net /CTS: now also J13.6 (Pin_6)
- net /DTR: no longer names the net of U3.4 (DTR#)
- net /DTR: now also J14.1 (Pin_1)
- net /RTS: no longer names the net of U3.6 (RTS#)
- net /RTS: now also J13.5 (Pin_5)
- new net: C19.2, J15.3 (Pin_3), U2.1 (Vout)
- new net: J12.1 (Pin_1), J13.4 (Pin_4), J15.2 (Pin_2)
- no-connect marks 0 -> 1
