File: STEP_TACHO/StepDriver/StepDriver.kicad_sch (KiCad schematic)
At the start: 15 parts, among them J1 STEP-MOTOR, J2 H:0.5V/L:0.125V, J3 M1, J4 M2, J5 DCY, J6 I/F, J7 POWER, U1 TB6608FNG

Commit message: Update: cleanup
Parts:
- added H1, H2, H3, H4: 3mm, KiCAD_lib:Hole3mm, symbol akizuki:Hole3mm
Changed lines of the file:
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@@
+    )
+  )
+  (symbol (lib_id "akizuki:Hole3mm") (at 66.04 69.85 0) (unit 1)
+    (in_bom yes) (on_board yes) (dnp no) (fields_autoplaced)
+    (property "Reference" "H4" (at 67.945 69.2063 0)
+      (effects (font (size 1.27 1.27)) (justify left))
+    )
+    (property "Value" "3mm" (at 67.945 71.1273 0)
+      (effects (font (size 1.27 1.27)) (justify left))
+    )
+    (property "Footprint" "KiCAD_lib:Hole3mm" (at 66.04 72.39 0)
+      (effects (font (size 1.27 1.27)) hide)
+    )
+    (property "Datasheet" "" (at 66.04 69.85 0)
+      (effects (font (size 1.27 1.27)) hide)
+    )
+    (instances
+      (project "StepDriver"
+        (path "/fe6068e1-55db-4f20-8000-579213a216a3"
+          (reference "H4") (unit 1)
+        )
+      )
     )
   )
@@
     )
   )
+  (symbol (lib_id "akizuki:Hole3mm") (at 66.04 39.37 0) (unit 1)
+    (in_bom yes) (on_board yes) (dnp no) (fields_autoplaced)
+    (property "Reference" "H1" (at 67.945 38.7263 0)
+      (effects (font (size 1.27 1.27)) (justify left))
+    )
+    (property "Value" "3mm" (at 67.945 40.6473 0)
+      (effects (font (size 1.27 1.27)) (justify left))
+    )
+    (property "Footprint" "KiCAD_lib:Hole3mm" (at 66.04 41.91 0)
+      (effects (font (size 1.27 1.27)) hide)
+    )
+    (property "Datasheet" "" (at 66.04 39.37 0)
+      (effects (font (size 1.27 1.27)) hide)
+    )
+    (instances
+      (project "StepDriver"
+        (path "/fe6068e1-55db-4f20-8000-579213a216a3"
+          (reference "H1") (unit 1)
+        )
+      )
+    )
+  )
+  (symbol (lib_id "akizuki:Hole3mm") (at 66.04 49.53 0) (unit 1)
+    (in_bom yes) (on_board yes) (dnp no) (fields_autoplaced)
+    (property "Reference" "H2" (at 67.945 48.8863 0)
+      (effects (font (size 1.27 1.27)) (justify left))
+    )
+    (property "Value" "3mm" (at 67.945 50.8073 0)
+      (effects (font (size 1.27 1.27)) (justify left))
+    )
+    (property "Footprint" "KiCAD_lib:Hole3mm" (at 66.04 52.07 0)
+      (effects (font (size 1.27 1.27)) hide)
+    )
+    (property "Datasheet" "" (at 66.04 49.53 0)
+      (effects (font (size 1.27 1.27)) hide)
+    )
+    (instances
+      (project "StepDriver"
+        (path "/fe6068e1-55db-4f20-8000-579213a216a3"
+          (reference "H2") (unit 1)
+        )
+      )
+    )
+  )
   (symbol (lib_id "akizuki:C-POL") (at 195.58 55.88 0) (unit 1)
     (in_bom yes) (on_board yes) (dnp no) (fields_autoplaced)
@@
         )
       )
+    )
+  )
+  (symbol (lib_id "akizuki:Hole3mm") (at 66.04 59.69 0) (unit 1)
+    (in_bom yes) (on_board yes) (dnp no) (fields_autoplaced)
+    (property "Reference" "H3" (at 67.945 59.0463 0)
+      (effects (font (size 1.27 1.27)) (justify left))
+    )
+    (property "Value" "3mm" (at 67.945 60.9673 0)
+      (effects (font (size 1.27 1.27)) (justify left))
+    )
+    (property "Footprint" "KiCAD_lib:Hole3mm" (at 66.04 62.23 0)
+      (effects (font (size 1.27 1.27)) hide)
+    )
+    (property "Datasheet" "" (at 66.04 59.69 0)
+      (effects (font (size 1.27 1.27)) hide)
+    )
+    (instances
+      (project "StepDriver"
+        (path "/fe6068e1-55db-4f20-8000-579213a216a3"
+          (reference "H3") (unit 1)
+        )
+      )
