File: rxprog/USB_CH9102F/USB_CH9102F.kicad_pcb (KiCad board)
At the start: 2 copper layers, 69 x 29 mm, 26 parts, among them J1 5077CR-16-SMC2-BK-TR, J2 USB/OPT, J3 Serial In/Out Full, J4 GPIO, J5 SUSPEND, J6 /SUSPEND, J7 /ACT, J8 /RST, J9 Serial In/Out, SW1 3P-SW, U1 CH9102F, U2 NJU7223DL1-33

Commit message: Update: sch/pcb
Parts:
- added H1: ~, KiCAD_lib:Hole3.2mm, F.Cu at (93.2, 83.3)
- added H2: ~, KiCAD_lib:Hole3.2mm, F.Cu at (156.7, 83.3)
- added H3: ~, KiCAD_lib:Hole3.2mm, F.Cu at (156.7, 106.8)
- added H4: ~, KiCAD_lib:Hole3.2mm, F.Cu at (93.2, 106.8)
- C4: value 4,7uF -> 10uF
- moved J1 0.50 mm to (92.5, 95.0)
Routing:
- net Net-(U1-D-): track 10.8 -> 12.7 mm
- net Net-(J1-SBU1): track 12.5 -> 13.5 mm, vias 0 -> 2
Other:
- board size 69 x 29 mm -> 70.4 x 29.6 mm
- board text added: "TAKACHI CS75N"
