File: rxprog/USB_CH9102F/USB_CH9102F.kicad_pcb (KiCad board)
At the start: 2 copper layers, 70.4 x 29.6 mm, 30 parts, among them J1 5077CR-16-SMC2-BK-TR, J2 USB/OPT, J3 Serial In/Out Full, J4 GPIO, J5 SUSPEND, J6 /SUSPEND, J7 /ACT, J8 /RST, J9 Serial In/Out, SW1 3P-SW, U1 CH9102F, U2 NJU7223DL1-33

Commit message: Update: cleanup
Routing:
- net +5V: track 63.9 -> 65.2 mm
Changed lines of the file:
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@@
 		(grid_origin 150 95)
 		(pcbplotparams
-			(layerselection 0x00000000_00000000_555555d5_575555f0)
+			(layerselection 0x00000000_00000000_555555d5_5755f5ff)
 			(plot_on_all_layers_selection 0x00000000_00000000_00000000_00000000)
 			(disableapertmacros no)
@@
 			(crossoutdnponfab yes)
 			(subtractmaskfromsilk no)
-			(outputformat 4)
+			(outputformat 1)
 			(mirror no)
 			(drillshape 0)
@@
 		)
 	)
+	(gr_arc
+		(start 89.961532 84.600012)
+		(mid 90.894122 81.878086)
+		(end 93.3 80.3)
+		(stroke
+			(width 0.1)
+			(type default)
+		)
+		(layer "F.SilkS")
+	)
+	(gr_arc
+		(start 93.299996 109.699986)
+		(mid 90.894125 108.121898)
+		(end 89.961528 105.399974)
+		(stroke
+			(width 0.1)
+			(type default)
+		)
+		(layer "F.SilkS")
+	)
+	(gr_arc
+		(start 156.699957 80.399972)
+		(mid 159.105835 81.978058)
+		(end 160.038425 84.699984)
+		(stroke
+			(width 0.1)
+			(type default)
+		)
+		(layer "F.SilkS")
+	)
+	(gr_arc
+		(start 160.038468 105.399988)
+		(mid 159.105878 108.121914)
+		(end 156.7 109.7)
+		(stroke
+			(width 0.1)
+			(type default)
+		)
+		(layer "F.SilkS")
+	)
 	(gr_line
 		(start 89.8 80.2)
@@
 	)
 	(segment
-		(start 106.05 96.9375)
-		(end 105.55 96.9375)
-		(width 0.2)
-		(layer "F.Cu")
-		(net "+5V")
-	)
-	(segment
 		(start 105.55 96.9375)
 		(end 105.55 98.5875)
@@
 	)
 	(segment
+		(start 106.05 98.0875)
+		(end 105.55 98.5875)
+		(width 0.2)
+		(layer "F.Cu")
+		(net "+5V")
+	)
+	(segment
 		(start 127.3 82)
 		(end 109.16 82)
@@
 	)
 	(segment
+		(start 106.05 96.9375)
+		(end 106.05 98.0875)
+		(width 0.2)
+		(layer "F.Cu")
+		(net "+5V")
+	)
+	(segment
 		(start 102.4875 88.6725)
 		(end 106.16 85)
@@
 	)
 	(segment
-		(start 108.7375 96.25)
-		(end 108.862499 96.374999)
+		(start 121.65 96.25)
+		(end 121.7 96.2)
 		(width 0.2)
 		(layer "F.Cu")
@@
 	)
 	(segment
-		(start 108.862499 96.374999)
-		(end 121.525001 96.374999)
-		(width 0.2)
-		(layer "F.Cu")
-		(net "Net-(J4-Pin_2)")
-	)
-	(segment
-		(start 121.525001 96.374999)
-		(end 121.7 96.2)
+		(start 108.7375 96.25)
+		(end 121.65 96.25)
 		(width 0.2)
 		(layer "F.Cu")

Commit message: Update: cleanup
Parts:
- C1: value 1uF -> 10uF
Changed lines of the file:
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@@
 			)
 		)
-		(property "Value" "1uF"
-			(at 0 1.43 0)
+		(property "Value" "10uF"
+			(at 0 -1.5 0)
 			(layer "F.Fab")
 			(effects

Commit message: Update: cleanup
Parts:
- moved D1 22.1 mm to (151.4, 83.9), turned to 180 degrees
- moved R1 16.8 mm to (146.4, 83.9)
Routing:
- net +5V: track 65.2 -> 84.2 mm, vias 4 -> 3
- net GND: track 40.6 -> 22.5 mm, vias 44 -> 42
- net Net-(D1-A): track 4.66 -> 3.06 mm, vias 2 -> 0
- net //DSR: track 45.7 -> 44.6 mm
- net //DTR: track 50.3 -> 49.7 mm
Other:
- board text added: "CH9102F"
