File: rxprog/USB_CH9102F/USB_CH9102F.kicad_sch (KiCad schematic)
At the start: 30 parts, among them J1 5077CR-16-SMC2-BK-TR, J2 USB/OPT, J3 Serial In/Out Full, J4 GPIO, J5 SUSPEND, J6 /SUSPEND, J7 /ACT, J8 /RST, J9 Serial In/Out, SW1 3P-SW, U1 CH9102F, U2 NJU7223DL1-33

Commit message: Update: cleanup
Parts:
- C1: value 1uF -> 10uF
Changed lines of the file:
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@@
 			)
 		)
-		(property "Value" "1uF"
+		(property "Value" "10uF"
 			(at 71.882 77.6164 0)
 			(show_name no)
